Commit message: WIP: fixing wrist images not showing up

File: aic_description/urdf/ur_gz.urdf.xacro (robot description, xacro)
@@ -144,4 +144,28 @@
     >
   </xacro:basler_camera>
+  <xacro:basler_camera
+    name="overview_camera"
+    tf_prefix="overview_camera/"
+    use_sim_cam="$(arg use_sim_cam)"
+    >
+  </xacro:basler_camera>
+  <xacro:basler_camera
+    name="overview_front_camera"
+    tf_prefix="overview_front_camera/"
+    use_sim_cam="$(arg use_sim_cam)"
+    >
+  </xacro:basler_camera>
+  <xacro:basler_camera
+    name="overview_side_camera"
+    tf_prefix="overview_side_camera/"
+    use_sim_cam="$(arg use_sim_cam)"
+    >
+  </xacro:basler_camera>
+  <xacro:basler_camera
+    name="overview_oblique_camera"
+    tf_prefix="overview_oblique_camera/"
+    use_sim_cam="$(arg use_sim_cam)"
+    >
+  </xacro:basler_camera>
   <xacro:robotiq_hande
     name="gripper"
@@ -188,4 +212,24 @@
     <parent link="$(arg cam_mount_tf_prefix)cam_mount_link"/>
     <child link="$(arg right_camera_tf_prefix)camera_link"/>
+  </joint>
+  <joint name="attach_overview_camera" type="fixed">
+    <origin xyz="-1.149822 0.300681 0.16" rpy="0 0 -0.00218531"/>
+    <parent link="tabletop"/>
+    <child link="overview_camera/camera_link"/>
+  </joint>
+  <joint name="attach_overview_front_camera" type="fixed">
+    <origin xyz="-0.349259 1.250207 0.08" rpy="1.5708 0 -1.57138531"/>
+    <parent link="tabletop"/>
+    <child link="overview_front_camera/camera_link"/>
+  </joint>
+  <joint name="attach_overview_side_camera" type="fixed">
+    <origin xyz="0.750207 0.349555 0.04" rpy="0 0 3.141"/>
+    <parent link="tabletop"/>
+    <child link="overview_side_camera/camera_link"/>
+  </joint>
+  <joint name="attach_overview_oblique_camera" type="fixed">
+    <origin xyz="-1.149318 1.150681 0.41" rpy="0 0 -0.79218531"/>
+    <parent link="tabletop"/>
+    <child link="overview_oblique_camera/camera_link"/>
   </joint>
   <joint name="attach_gripper" type="fixed">

Commit message: checkpoint for working VLM based trajectory generation. Current score is low, timestep is large (~100) although videos are being saved

File: aic_description/urdf/ur_gz.urdf.xacro (robot description, xacro)
@@ -144,28 +144,4 @@
     >
   </xacro:basler_camera>
-  <xacro:basler_camera
-    name="overview_camera"
-    tf_prefix="overview_camera/"
-    use_sim_cam="$(arg use_sim_cam)"
-    >
-  </xacro:basler_camera>
-  <xacro:basler_camera
-    name="overview_front_camera"
-    tf_prefix="overview_front_camera/"
-    use_sim_cam="$(arg use_sim_cam)"
-    >
-  </xacro:basler_camera>
-  <xacro:basler_camera
-    name="overview_side_camera"
-    tf_prefix="overview_side_camera/"
-    use_sim_cam="$(arg use_sim_cam)"
-    >
-  </xacro:basler_camera>
-  <xacro:basler_camera
-    name="overview_oblique_camera"
-    tf_prefix="overview_oblique_camera/"
-    use_sim_cam="$(arg use_sim_cam)"
-    >
-  </xacro:basler_camera>
   <xacro:robotiq_hande
     name="gripper"
@@ -212,24 +188,4 @@
     <parent link="$(arg cam_mount_tf_prefix)cam_mount_link"/>
     <child link="$(arg right_camera_tf_prefix)camera_link"/>
-  </joint>
-  <joint name="attach_overview_camera" type="fixed">
-    <origin xyz="-1.149822 0.300681 0.16" rpy="0 0 -0.00218531"/>
-    <parent link="tabletop"/>
-    <child link="overview_camera/camera_link"/>
-  </joint>
-  <joint name="attach_overview_front_camera" type="fixed">
-    <origin xyz="-0.349259 1.250207 0.08" rpy="1.5708 0 -1.57138531"/>
-    <parent link="tabletop"/>
-    <child link="overview_front_camera/camera_link"/>
-  </joint>
-  <joint name="attach_overview_side_camera" type="fixed">
-    <origin xyz="0.750207 0.349555 0.04" rpy="0 0 3.141"/>
-    <parent link="tabletop"/>
-    <child link="overview_side_camera/camera_link"/>
-  </joint>
-  <joint name="attach_overview_oblique_camera" type="fixed">
-    <origin xyz="-1.149318 1.150681 0.41" rpy="0 0 -0.79218531"/>
-    <parent link="tabletop"/>
-    <child link="overview_oblique_camera/camera_link"/>
   </joint>
   <joint name="attach_gripper" type="fixed">
